File: Hardware/HAR_Board/HAR_Board.sch (KiCad schematic (older format))
At the start: 0 parts

Commit message: Initial HW files
Parts:
- added P?: USB_C_Plug_USB2.0, symbol Connector:USB_C_Plug_USB2.0
Connections:
- new net: P?.A1 (GND), P?.A12 (GND), P?.B1 (GND), P?.B12 (GND)
- new net: P?.A4 (VBUS), P?.A9 (VBUS), P?.B4 (VBUS), P?.B9 (VBUS)
Changed lines of the file:
@@
 Comment4 ""
 $EndDescr
+$Comp
+L Connector:USB_C_Plug_USB2.0 P?
+U 1 1 61574032
+P 2400 2600
+F 0 "P?" H 2507 3467 50  0000 C CNN
+F 1 "USB_C_Plug_USB2.0" H 2507 3376 50  0000 C CNN
+F 2 "" H 2550 2600 50  0001 C CNN
+F 3 "https://www.usb.org/sites/default/files/documents/usb_type-c.zip" H 2550 2600 50  0001 C CNN
+	1    2400 2600
+	1    0    0    -1
+$EndComp
 $EndSCHEMATC
