File: Hardware/HAR_Board/CluePCB.kicad_pcb (KiCad board)
At the start: 2 copper layers, 78.7 x 76.2 mm, 8 parts, among them M3 MountingHole, U1 LoRa, U2 GPS, U3 Dragontail, U4 PowerBoost500

Commit message: Add files via upload
New voltage divider changes
Parts:
- added R1: 2.2k, Resistor_THT:R_Axial_DIN0204_L3.6mm_D1.6mm_P5.08mm_Horizontal, F.Cu at (162.6, 70.4)
- added R2: 3.3k, Resistor_THT:R_Axial_DIN0204_L3.6mm_D1.6mm_P5.08mm_Horizontal, F.Cu at (153.5, 70.4)
- added U5: Drag3V, HABET_Lib:Dragon3V, F.Cu at (135.9, 84.2)
- moved M3 7.47 mm to (144.5, 93.5)
- moved M3 5.00 mm to (206.2, 90.9)
- moved U4 4.58 mm to (187.9, 74.4)
Connections:
- U4 pad 3: unconnected-(U4-Pad3) -> Net-(R1-Pad2)
Routing:
- net Net-(R1-Pad1): track 0.00 -> 9.09 mm
- net Net-(R1-Pad2): track 0.00 -> 5.36 mm
- removed copper zone on F.Cu, net Net-(U1-Pad1)
Other:
- board size 78.7 x 76.2 mm -> 78.7 x 81.3 mm
