File: pcb/CluePCB.kicad_pcb (KiCad board)
At the start: 2 copper layers, 168.4 x 113.3 mm, 16 parts, among them J1 Conn_01x02, J2 Conn_01x02, J3 Conn_01x02, M3MM-1 MountingHole_3mm, M3MM-2 MountingHole_3mm, M3MM-3 MountingHole_3mm, SW1 SW_SPST, U1 Sparkfun_PRT-14411, U2 INA219-BOB, U3 AZ1117-3.3, U4 Sparkfun_Microbit_BOB-16446, U5 Adafruit_RFM96W-3073, U6 Sparkfun_GPS_NEO-M9N

Commit message: Generated Gerber files
Final update, generated gerber files
Parts:
- removed M3MM-1, M3MM-2, M3MM-3: MountingHole_3mm, MountingHole:MountingHole_3mm
- added H1: MountingHole, MountingHole:MountingHole_3mm, F.Cu at (66.3, 140.0)
- added H2: MountingHole, MountingHole:MountingHole_3mm, F.Cu at (66.4, 42.0)
- added H3: MountingHole, MountingHole:MountingHole_3mm, F.Cu at (221.8, 138.9)
- moved J1 95.3 mm to (64.1, 50.2)
- moved J2 78.2 mm to (112.5, 67.0), turned to -90 degrees
- moved U5 34.6 mm to (211.8, 100.7)
Connections:
- net Net-(U4-Pad12) renamed G0
- net Net-(U4-Pad17) renamed SCK
- net Net-(U4-Pad18) renamed MISO
- net Net-(U4-Pad19) renamed MOSI
- net Net-(U4-Pad20) renamed CS
- net Net-(U4-Pad6) renamed RST
Routing:
- net Net-(J2-Pad2): track 128.4 -> 27.2 mm
- net +5V: track 100.8 -> 32.0 mm
- net GND: track 18.4 -> 45.7 mm
- net MOSI: track 54.8 -> 29.3 mm
- net MISO: track 57.4 -> 32.9 mm
- net CS: track 49.8 -> 26.7 mm
- net SCK: track 56.2 -> 37.5 mm
- net G0: track 66.3 -> 50.3 mm
- net RST: track 72.5 -> 61.6 mm
Other:
- board size 168.4 x 113.3 mm -> 168.4 x 109.6 mm
- board text added: "Clue Board"
- board text added: "GPS Module"
- board text added: "High Altitude Reporter (HAR) Rev 1.0 Matthew Nelson"
- board text added: "LoRa Module"
- board text added: "PWR MON"
- board text added: "PWR Module"

Commit message: Fabrication run
Other:
- board text added: "High Altitude Reporter (HAR) Gen3 Rev 1.0 Matthew Nelson"
- board text removed: "High Altitude Reporter (HAR) Rev 1.0 Matthew Nelson"
