File: pcb/CluePCB.kicad_sch (KiCad schematic)
At the start: 13 parts, among them J1 Conn_01x02, J2 Conn_01x02, J3 Conn_01x02, SW1 SW_SPST, U1 Sparkfun_PRT-14411, U2 INA219-BOB, U3 AZ1117-3.3, U4 Sparkfun_Microbit_BOB-16446, U5 Adafruit_RFM96W-3073, U6 Sparkfun_GPS_NEO-M9N

Commit message: Generated Gerber files
Final update, generated gerber files
Parts:
- added H1, H2, H3: MountingHole, MountingHole:MountingHole_3mm, symbol Mechanical:MountingHole
Connections:
- net G0: now reaches U4.12 (GP), U5.4 (G0)
- net SCK: now reaches U4.17 (SCK), U5.5 (SCK)
- net MISO: now reaches U4.18 (MISO), U5.6 (MISO)
- net MOSI: now reaches U4.19 (MOSI), U5.7 (MOSI)
- net CS: now reaches U4.20 (GP16), U5.8 (CS)
- net RST: now reaches U4.6 (AIN2), U5.9 (RST)
Changed lines of the file:
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@@
     (stroke (width 0) (type default) (color 0 0 0 0))
+  )
+  (global_label "CS" (shape input) (at 196.85 69.85 0) (fields_autoplaced)
+    (effects (font (size 1.27 1.27)) (justify left))
+    (property "Intersheet References" "${INTERSHEET_REFS}" (id 0) (at 201.7426 69.7706 0)
+      (effects (font (size 1.27 1.27)) (justify left) hide)
+    )
+  )
+  (global_label "MISO" (shape input) (at 191.77 74.93 180) (fields_autoplaced)
+    (effects (font (size 1.27 1.27)) (justify right))
+    (property "Intersheet References" "${INTERSHEET_REFS}" (id 0) (at 184.7607 74.8506 0)
+      (effects (font (size 1.27 1.27)) (justify right) hide)
+    )
+  )
+  (global_label "SCK" (shape input) (at 189.23 69.85 180) (fields_autoplaced)
+    (effects (font (size 1.27 1.27)) (justify right))
+    (property "Intersheet References" "${INTERSHEET_REFS}" (id 0) (at 183.0674 69.7706 0)
+      (effects (font (size 1.27 1.27)) (justify right) hide)
+    )
+  )
+  (global_label "MOSI" (shape input) (at 194.31 80.01 180) (fields_autoplaced)
+    (effects (font (size 1.27 1.27)) (justify right))
+    (property "Intersheet References" "${INTERSHEET_REFS}" (id 0) (at 187.3007 79.9306 0)
+      (effects (font (size 1.27 1.27)) (justify right) hide)
+    )
+  )
+  (global_label "RST" (shape input) (at 161.29 72.39 0) (fields_autoplaced)
+    (effects (font (size 1.27 1.27)) (justify left))
+    (property "Intersheet References" "${INTERSHEET_REFS}" (id 0) (at 167.1502 72.3106 0)
+      (effects (font (size 1.27 1.27)) (justify left) hide)
+    )
+  )
+  (global_label "G0" (shape input) (at 176.53 72.39 180) (fields_autoplaced)
+    (effects (font (size 1.27 1.27)) (justify right))
+    (property "Intersheet References" "${INTERSHEET_REFS}" (id 0) (at 171.6374 72.3106 0)
+      (effects (font (size 1.27 1.27)) (justify right) hide)
+    )
   )
   (symbol (lib_id "power:+5V") (at 57.15 99.06 0) (unit 1)
@@
   (symbol (lib_id "power:+3V3") (at 160.02 99.06 0) (unit 1)
     (in_bom yes) (on_board yes) (fields_autoplaced)
-    (property "Reference" "#PWR0101" (id 0) (at 160.02 102.87 0)
+    (property "Reference" "#PWR06" (id 0) (at 160.02 102.87 0)
       (effects (font (size 1.27 1.27)) hide)
     )
@@
     (pin "9")
   )
+  (symbol (lib_id "Mechanical:MountingHole") (at 30.48 35.56 0) (unit 1)
+    (in_bom yes) (on_board yes) (fields_autoplaced)
+    (property "Reference" "H2" (id 0) (at 33.02 34.2899 0)
+      (effects (font (size 1.27 1.27)) (justify left))
+    )
+    (property "Value" "MountingHole" (id 1) (at 33.02 36.8299 0)
+      (effects (font (size 1.27 1.27)) (justify left))
+    )
+    (property "Footprint" "MountingHole:MountingHole_3mm" (id 2) (at 30.48 35.56 0)
+      (effects (font (size 1.27 1.27)) hide)
+    )
+    (property "Datasheet" "~" (id 3) (at 30.48 35.56 0)
+      (effects (font (size 1.27 1.27)) hide)
+    )
+  )
   (symbol (lib_id "Regulator_Linear:AZ1117-3.3") (at 142.24 99.06 0) (unit 1)
     (in_bom yes) (on_board yes) (fields_autoplaced)
@@
     (pin "2")
     (pin "3")
+  )
+  (symbol (lib_id "Mechanical:MountingHole") (at 48.26 22.86 0) (unit 1)
+    (in_bom yes) (on_board yes) (fields_autoplaced)
+    (property "Reference" "H3" (id 0) (at 50.8 21.5899 0)
+      (effects (font (size 1.27 1.27)) (justify left))
+    )
+    (property "Value" "MountingHole" (id 1) (at 50.8 24.1299 0)
+      (effects (font (size 1.27 1.27)) (justify left))
+    )
+    (property "Footprint" "MountingHole:MountingHole_3mm" (id 2) (at 48.26 22.86 0)
+      (effects (font (size 1.27 1.27)) hide)
+    )
+    (property "Datasheet" "~" (id 3) (at 48.26 22.86 0)
+      (effects (font (size 1.27 1.27)) hide)
+    )
   )
   (symbol (lib_id "power:GND") (at 62.23 91.44 0) (unit 1)
@@
     (pin "1")
   )
+  (symbol (lib_id "Mechanical:MountingHole") (at 30.48 22.86 0) (unit 1)
+    (in_bom yes) (on_board yes) (fields_autoplaced)
+    (property "Reference" "H1" (id 0) (at 33.02 21.5899 0)
+      (effects (font (size 1.27 1.27)) (justify left))
+    )
+    (property "Value" "MountingHole" (id 1) (at 33.02 24.1299 0)
+      (effects (font (size 1.27 1.27)) (justify left))
+    )
+    (property "Footprint" "MountingHole:MountingHole_3mm" (id 2) (at 30.48 22.86 0)
+      (effects (font (size 1.27 1.27)) hide)
+    )
+    (property "Datasheet" "~" (id 3) (at 30.48 22.86 0)
+      (effects (font (size 1.27 1.27)) hide)
+    )
+  )
   (sheet_instances
     (path "/" (page "1"))
@@
     )
     (path "/45746010-0fb1-4548-9da6-cb3f04f25368"
-      (reference "#PWR0101") (unit 1) (value "+3V3") (footprint "")
+      (reference "#PWR06") (unit 1) (value "+3V3") (footprint "")
     )
     (path "/00cba8a2-a55e-474a-8579-54c3cf8b08cf"
@@
       (reference "C2") (unit 1) (value "0.1uF") (footprint "Capacitor_THT:C_Rect_L7.0mm_W4.5mm_P5.00mm")
     )
+    (path "/ee13e400-85d6-4977-a3f5-32c2817b13b9"
+      (reference "H1") (unit 1) (value "MountingHole") (footprint "MountingHole:MountingHole_3mm")
+    )
+    (path "/566cafa1-3861-4a6e-9f7b-93d1942825df"
+      (reference "H2") (unit 1) (value "MountingHole") (footprint "MountingHole:MountingHole_3mm")
+    )
+    (path "/5d400caa-fa72-44a0-acf3-6b3fad565c32"
+      (reference "H3") (unit 1) (value "MountingHole") (footprint "MountingHole:MountingHole_3mm")
+    )
     (path "/b5fcd6a2-d55f-45e3-b876-86893b8abf02"
